File: PCBs/learsim pcbs.kicad_sch (KiCad schematic)
At the start: 51 parts, among them SW1 MHz, SW2 KHz, U1 ESP32-C6-DEV-KIT-N8, U2 MAX7219, U3 MAX7219

Commit message: Add new toggle switch symbol and footprint for 1FS1T1B9M2RES-5
- Created a new symbol for the toggle switch 1FS1T1B9M2RES-5 in the easyeda2kicad library, including properties such as reference, value, footprint, datasheet, manufacturer, MPN, and LCSC part number.
- Added a corresponding footprint module for the toggle switch, defining pads, silk screen, and 3D model for better visualization in PCB design.
Parts:
- added SW3: 1FS1T1B9M2RES-5, Rotary:SW-TH_1FS1T1B9M2RES-5, symbol Rotary:1FS1T1B9M2RES-5
Changed lines of the file:
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@@
+	)
+	(symbol
+		(lib_id "Rotary:1FS1T1B9M2RES-5")
+		(at 35.56 72.39 0)
+		(unit 1)
+		(body_style 1)
+		(exclude_from_sim no)
+		(in_bom yes)
+		(on_board yes)
+		(in_pos_files yes)
+		(dnp no)
+		(fields_autoplaced yes)
+		(property "Reference" "SW3"
+			(at 41.91 69.2149 0)
+			(show_name no)
+			(do_not_autoplace no)
+			(effects
+				(font
+					(size 1.27 1.27)
+				)
+				(justify left)
+			)
+		)
+		(property "Value" "1FS1T1B9M2RES-5"
+			(at 41.91 71.7549 0)
+			(show_name no)
+			(do_not_autoplace no)
+			(effects
+				(font
+					(size 1.27 1.27)
+				)
+				(justify left)
+			)
+		)
+		(property "Footprint" "Rotary:SW-TH_1FS1T1B9M2RES-5"
+			(at 35.56 85.09 0)
+			(hide yes)
+			(show_name no)
+			(do_not_autoplace no)
+			(effects
+				(font
+					(size 1.27 1.27)
+				)
+			)
+		)
+		(property "Datasheet" "https://lcsc.com/product-detail/New-Arrivals_Dailywell-1FS1T1B9M2RES-5_C496164.html"
+			(at 35.56 87.63 0)
+			(hide yes)
+			(show_name no)
+			(do_not_autoplace no)
+			(effects
+				(font
+					(size 1.27 1.27)
+				)
+			)
+		)
+		(property "Description" ""
+			(at 35.56 72.39 0)
+			(hide yes)
+			(show_name no)
+			(do_not_autoplace no)
+			(effects
+				(font
+					(size 1.27 1.27)
+				)
+			)
+		)
+		(property "Manufacturer" "Dailywell(德利威)"
+			(at 35.56 90.17 0)
+			(hide yes)
+			(show_name no)
+			(do_not_autoplace no)
+			(effects
+				(font
+					(size 1.27 1.27)
+				)
+			)
+		)
+		(property "MPN" "1FS1T1B9M2RES-5"
+			(at 35.56 92.71 0)
+			(hide yes)
+			(show_name no)
+			(do_not_autoplace no)
+			(effects
+				(font
+					(size 1.27 1.27)
+				)
+			)
+		)
+		(property "LCSC Part" "C496164"
+			(at 35.56 95.25 0)
+			(hide yes)
+			(show_name no)
+			(do_not_autoplace no)
+			(effects
+				(font
+					(size 1.27 1.27)
+				)
+			)
+		)
+		(pin "3"
+		)
+		(pin "2"
+		)
+		(pin "1"
+		)
+		(instances
+			(project "learsim pcbs"
+				(path "/27520048-f2d9-41fa-a766-14782a208ac0"
+					(reference "SW3")
+					(unit 1)
+				)
+			)
+		)
 	)
 	(symbol

Commit message: Add new toggle switch symbols and footprints for 2MD3T1B1M2QES-5 and 2MS1T1B1M2QES-5
- Created symbol for 2MD3T1B1M2QES-5 with properties including reference, value, footprint, datasheet, manufacturer, MPN, and LCSC part.
- Added graphical representation including pins and connections for 2MD3T1B1M2QES-5.
- Created symbol for 2MS1T1B1M2QES-5 with similar properties and graphical representation.
- Added corresponding footprints for both switches in the KiCad library.
Parts:
- removed SW3: 1FS1T1B9M2RES-5, Rotary:SW-TH_1FS1T1B9M2RES-5, symbol Rotary:1FS1T1B9M2RES-5
- added SW3: 2MS1T1B1M2QES-5, Rotary:SW-TH_2MS1T1B1M2QES-5, symbol Rotary:2MS1T1B1M2QES-5
Connections:
- net U2_ISET: now also U2.18 (ISET); no longer U2.24 (DOUT)
Changed lines of the file:
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@@
 	(global_label "U2_ISET"
 		(shape bidirectional)
-		(at 90.17 125.73 90)
+		(at 49.53 146.05 270)
 		(fields_autoplaced yes)
 		(effects
@@
 				(size 1.27 1.27)
 			)
-			(justify left)
+			(justify right)
 		)
 		(property "Intersheetrefs" "${INTERSHEET_REFS}"
-			(at 90.17 114.195 90)
+			(at 49.53 157.585 90)
 			(hide yes)
 			(show_name no)
@@
 					(size 1.27 1.27)
 				)
-				(justify left)
+				(justify right)
 			)
 		)
@@
 	)
 	(symbol
-		(lib_id "Rotary:1FS1T1B9M2RES-5")
-		(at 35.56 72.39 0)
-		(unit 1)
-		(body_style 1)
-		(exclude_from_sim no)
-		(in_bom yes)
-		(on_board yes)
-		(in_pos_files yes)
-		(dnp no)
-		(fields_autoplaced yes)
-		(property "Reference" "SW3"
-			(at 41.91 69.2149 0)
-			(show_name no)
-			(do_not_autoplace no)
-			(effects
-				(font
-					(size 1.27 1.27)
-				)
-				(justify left)
-			)
-		)
-		(property "Value" "1FS1T1B9M2RES-5"
-			(at 41.91 71.7549 0)
-			(show_name no)
-			(do_not_autoplace no)
-			(effects
-				(font
-					(size 1.27 1.27)
-				)
-				(justify left)
-			)
-		)
-		(property "Footprint" "Rotary:SW-TH_1FS1T1B9M2RES-5"
-			(at 35.56 85.09 0)
-			(hide yes)
-			(show_name no)
-			(do_not_autoplace no)
-			(effects
-				(font
-					(size 1.27 1.27)
-				)
-			)
-		)
-		(property "Datasheet" "https://lcsc.com/product-detail/New-Arrivals_Dailywell-1FS1T1B9M2RES-5_C496164.html"
-			(at 35.56 87.63 0)
-			(hide yes)
-			(show_name no)
-			(do_not_autoplace no)
-			(effects
-				(font
-					(size 1.27 1.27)
-				)
-			)
-		)
-		(property "Description" ""
-			(at 35.56 72.39 0)
-			(hide yes)
-			(show_name no)
-			(do_not_autoplace no)
-			(effects
-				(font
-					(size 1.27 1.27)
-				)
-			)
-		)
-		(property "Manufacturer" "Dailywell(德利威)"
-			(at 35.56 90.17 0)
-			(hide yes)
-			(show_name no)
-			(do_not_autoplace no)
-			(effects
-				(font
-					(size 1.27 1.27)
-				)
-			)
-		)
-		(property "MPN" "1FS1T1B9M2RES-5"
-			(at 35.56 92.71 0)
-			(hide yes)
-			(show_name no)
-			(do_not_autoplace no)
-			(effects
-				(font
-					(size 1.27 1.27)
-				)
-			)
-		)
-		(property "LCSC Part" "C496164"
-			(at 35.56 95.25 0)
-			(hide yes)
-			(show_name no)
-			(do_not_autoplace no)
-			(effects
-				(font
-					(size 1.27 1.27)
-				)
-			)
-		)
-		(pin "3"
-		)
-		(pin "2"
-		)
-		(pin "1"
-		)
-		(instances
-			(project "learsim pcbs"
-				(path "/27520048-f2d9-41fa-a766-14782a208ac0"
-					(reference "SW3")
-					(unit 1)
-				)
-			)
-		)
-	)
-	(symbol
 		(lib_id "Device:C")
 		(at 290 91.12 0)
@@
 					(unit 1)
 				)
+			)
+		)
+	)
+	(symbol
+		(lib_id "Rotary:2MS1T1B1M2QES-5")
+		(at 24.13 48.26 0)
+		(unit 1)
+		(body_style 1)
+		(exclude_from_sim no)
+		(in_bom yes)
+		(on_board yes)
+		(in_pos_files yes)
+		(dnp no)
+		(fields_autoplaced yes)
+		(property "Reference" "SW3"
+			(at 29.21 46.9899 0)
+			(show_name no)
+			(do_not_autoplace no)
+			(effects
+				(font
+					(size 1.27 1.27)
+				)
+				(justify left)
+			)
+		)
+		(property "Value" "2MS1T1B1M2QES-5"
+			(at 29.21 49.5299 0)
+			(show_name no)
+			(do_not_autoplace no)
+			(effects
+				(font
+					(size 1.27 1.27)
+				)
+				(justify left)
+			)
+		)
+		(property "Footprint" "Rotary:SW-TH_2MS1T1B1M2QES-5"
+			(at 24.13 60.96 0)
+			(hide yes)
+			(show_name no)
+			(do_not_autoplace no)
+			(effects
+				(font
+					(size 1.27 1.27)
+				)
+			)
+		)
+		(property "Datasheet" "https://lcsc.com/product-detail/Toggle-Switches_Dailywell-2MS1T1B1M2QES-5_C908280.html"
+			(at 24.13 63.5 0)
+			(hide yes)
+			(show_name no)
+			(do_not_autoplace no)
+			(effects
+				(font
+					(size 1.27 1.27)
+				)
+			)
+		)
+		(property "Description" ""
+			(at 24.13 48.26 0)
+			(hide yes)
+			(show_name no)
+			(do_not_autoplace no)
+			(effects
+				(font
+					(size 1.27 1.27)
+				)
+			)
+		)
+		(property "Manufacturer" "Dailywell(德利威)"
+			(at 24.13 66.04 0)
+			(hide yes)
+			(show_name no)
+			(do_not_autoplace no)
+			(effects
+				(font
+					(size 1.27 1.27)
+				)
+			)
+		)
+		(property "MPN" "2MS1T1B1M2QES-5"
+			(at 24.13 68.58 0)
+			(hide yes)
+			(show_name no)
+			(do_not_autoplace no)
+			(effects
+				(font
+					(size 1.27 1.27)
+				)
+			)
+		)
+		(property "LCSC Part" "C908280"
+			(at 24.13 71.12 0)
+			(hide yes)
+			(show_name no)
+			(do_not_autoplace no)
+			(effects
+				(font
+					(size 1.27 1.27)
+				)
+			)
+		)
+		(pin "3"
+		)
+		(pin "2"
+		)
+		(pin "1"
+		)
+		(instances
+			(project "learsim pcbs"
+				(path "/27520048-f2d9-41fa-a766-14782a208ac0"
+					(reference "SW3")
+					(unit 1)
+				)

Commit message: Remove unused global labels and a capacitor symbol from the schematic. Adjust positions of rotary switch properties for better alignment.
Parts:
- removed C6: 100uF, Capacitor_THT:CP_Radial_D6.3mm_P2.50mm, symbol Device:C
Other:
- moved on the sheet: SW3

Commit message: Adjust positions of global labels in the schematic for better alignment
Connections:
- net MAX_CHAIN: now also U2.24 (DOUT); no longer U1.6 (GPIO6), U2.1 (DIN)
- new net SPI_DIN: U1.6 (GPIO6), U2.1 (DIN)
Changed lines of the file:
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@@
 	(global_label "MAX_CHAIN"
 		(shape bidirectional)
-		(at 90.17 146.05 0)
+		(at 90.17 125.73 0)
 		(fields_autoplaced yes)
 		(effects
@@
 		)
 		(property "Intersheetrefs" "${INTERSHEET_REFS}"
-			(at 104.608 146.05 0)
+			(at 104.608 125.73 0)
 			(hide yes)
 			(show_name no)

Commit message: Adjust global label positions and justification in the schematic for improved alignment
Connections:
- net +5V: now also U2.19 (V+), U3.19 (V+); no longer U2.4 (GND), U2.9 (GND), U3.4 (GND), U3.9 (GND)
- net GND: now also U2.4 (GND), U2.9 (GND), U3.4 (GND), U3.9 (GND); no longer U2.19 (V+), U3.19 (V+)
