File: PCBs/learsim pcbs.kicad_sch (KiCad schematic)
At the start: 53 parts, among them SW1 MHz, SW2 KHz, SW3 2MS1T1B1M2QES-5, U1 ESP32-C6-DEV-KIT-N8, U2 MAX7219, U3 MAX7219

Commit message: Move SW3 off ESP32-C6 boot pins; restore 5V bulk cap
Design-review fixes:
- SW3 was on GPIO8/GPIO9, both ESP32-C6 strapping pins (GPIO9 selects
  download boot). With the toggle common tied to GND, one position would
  hold GPIO9 low at reset and drop the board into download mode. Moved
  SW3 to boot-safe pins: pin1 -> GPIO14 (R15 pull-up), pin3 -> EXIO7
  (TCA9554 expander, R16 pull-up). GPIO8/GPIO9 are now spare.
- Restored a bulk reservoir cap C6 (220uF electrolytic) across +5V/GND at
  the J1 input for the display/LED current bursts.

Verified: SW3_A={SW3.1,R15,GPIO14}, SW3_B={SW3.3,R16,EXIO7}, C6 on +5V/GND,
0 floating pins, no shorts. README GPIO map/BOM updated.

Co-Authored-By: Claude Opus 4.8 <noreply@anthropic.com>
Claude-Session: https://claude.ai/code/session_01PYVnDFXSTkVYnSG662sK4G
Parts:
- added C6: 220uF, Capacitor_THT:CP_Radial_D6.3mm_P2.50mm, symbol Device:C
Connections:
- net +5V: now also C6.1
- net GND: now also C6.2
- net SW3_A: now also U1.8 (GPIO14); no longer U1.20 (GPIO8)
- net SW3_B: now also U1.15 (EXIO7); no longer U1.21 (GPIO9)
Changed lines of the file:
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@@
-		(effects (font (size 1.27 1.27)) (justify left))
-	)
-	(global_label "SW3_A"
-		(shape bidirectional)
-		(at 24.13 106.68 270)
-		(fields_autoplaced yes)
-		(effects (font (size 1.27 1.27)) (justify left))
-	)
-	(global_label "SW3_A"
-		(shape bidirectional)
-		(at 147.32 97.79 0)
-		(fields_autoplaced yes)
-		(effects (font (size 1.27 1.27)) (justify left))
-	)
-	(global_label "SW3_A"
-		(shape bidirectional)
-		(at 236.0 196.19 90)
-		(fields_autoplaced yes)
-		(effects (font (size 1.27 1.27)) (justify left))
-	)
-	(global_label "SW3_B"
-		(shape bidirectional)
-		(at 29.21 106.68 270)
-		(fields_autoplaced yes)
-		(effects (font (size 1.27 1.27)) (justify left))
-	)
-	(global_label "SW3_B"
-		(shape bidirectional)
-		(at 147.32 100.33 0)
-		(fields_autoplaced yes)
-		(effects (font (size 1.27 1.27)) (justify left))
-	)
-	(global_label "SW3_B"
-		(shape bidirectional)
-		(at 250.0 196.19 90)
-		(fields_autoplaced yes)
 		(effects (font (size 1.27 1.27)) (justify left))
 	)
@@
 		(fields_autoplaced yes)
 		(effects (font (size 1.27 1.27)) (justify left))
+	)
+	(symbol
+		(lib_id "Device:C")
+		(at 264.0 200.0 0)
+		(unit 1)
+		(body_style 1)
+		(exclude_from_sim no)
+		(in_bom yes)
+		(on_board yes)
+		(in_pos_files yes)
+		(dnp no)
+		(property "Reference" "C6"
+			(at 267.81 198.73 0)
+			(effects (font (size 1.27 1.27)) (justify left))
+		)
+		(property "Value" "220uF"
+			(at 267.81 201.27 0)
+			(effects (font (size 1.27 1.27)) (justify left))
+		)
+		(property "Footprint" "Capacitor_THT:CP_Radial_D6.3mm_P2.50mm"
+			(at 264.0 200.0 0)
+			(hide yes)
+			(effects (font (size 1.27 1.27)))
+		)
+		(property "Datasheet" "~"
+			(at 264.0 200.0 0)
+			(hide yes)
+			(effects (font (size 1.27 1.27)))
+		)
+		(pin "1"
+		)
+		(pin "2"
+		)
+		(instances
+			(project "learsim pcbs"
+				(path "/27520048-f2d9-41fa-a766-14782a208ac0"
+					(reference "C6")
+					(unit 1)
+				)
+			)
+		)
+	)
+	(global_label "SW3_A"
+		(shape bidirectional)
+		(at 24.13 106.68 270)
+		(fields_autoplaced yes)
+		(effects (font (size 1.27 1.27)) (justify left))
+	)
+	(global_label "SW3_A"
+		(shape bidirectional)
+		(at 236.0 196.19 90)
+		(fields_autoplaced yes)
+		(effects (font (size 1.27 1.27)) (justify left))
+	)
+	(global_label "SW3_A"
+		(shape bidirectional)
+		(at 111.76 105.41 180)
+		(fields_autoplaced yes)
+		(effects (font (size 1.27 1.27)) (justify left))
+	)
+	(global_label "SW3_B"
+		(shape bidirectional)
+		(at 29.21 106.68 270)
+		(fields_autoplaced yes)
+		(effects (font (size 1.27 1.27)) (justify left))
+	)
+	(global_label "SW3_B"
+		(shape bidirectional)
+		(at 250.0 196.19 90)
+		(fields_autoplaced yes)
+		(effects (font (size 1.27 1.27)) (justify left))
+	)
+	(global_label "SW3_B"
+		(shape bidirectional)
+		(at 111.76 123.19 270)
+		(fields_autoplaced yes)
+		(effects (font (size 1.27 1.27)) (justify left))
+	)
+	(global_label "+5V"
+		(shape bidirectional)
+		(at 264.0 196.19 90)
+		(fields_autoplaced yes)
+		(effects (font (size 1.27 1.27)) (justify left))
+	)
+	(global_label "GND"
+		(shape bidirectional)
+		(at 264.0 203.81 270)
+		(fields_autoplaced yes)
+		(effects (font (size 1.27 1.27)) (justify left))
