File: PCBs/learsim pcbs.kicad_pcb (KiCad board)
At the start: 2 copper layers, 120 x 110 mm, 58 parts, among them SW1 MHz, SW2 KHz, SW3 2MD1T1B1M2QES-5, U1 ESP32-C6-DEV-KIT-N8, U2 MAX7219, U3 MAX7219

Commit message: Update PCB files with new creation date and modify drill and aperture definitions
- Updated creation date in Gerber files (F_Mask, F_Paste, F_Silkscreen) to 2026-07-27.
- Adjusted aperture definitions in F_Mask for better alignment with design specifications.
- Refined drill files (NPTH and PTH) with updated creation date and corrected tool definitions.
- Enhanced job file with new creation date for consistency across project files.
Connections:
- U1 pad 11: SW3_A -> unconnected-(U1-GPIO8-Pad11)
- U1 pad 12: SW3_B -> unconnected-(U1-GPIO9-Pad12)
- U1 pad 19: unconnected-(U1-EXIO6-Pad19) -> SW3_A
- U1 pad 20: unconnected-(U1-EXIO7-Pad20) -> SW3_B
Routing:
- net SW3_A: track 82.6 -> 47.8 mm
- net SW3_B: track 80.7 -> 65.4 mm, vias 2 -> 0
- net +5V: track 476.0 -> 469.3 mm
- net +3V3: track 349.9 -> 356.2 mm, vias 2 -> 4
- net GND: track 94.7 -> 89.1 mm, vias 19 -> 17
- net SPI_LOAD: track 101.4 -> 102.0 mm
- net unconnected-(U1-GPIO8-Pad11): track 0.00 -> 0.56 mm

Commit message: v1.0
Parts:
- moved C4 120.7 mm to (26.2, 56.9), turned to 0 degrees
- moved C2 87.7 mm to (89.8, 47.9), turned to 180 degrees
- moved C6 82.2 mm to (122.8, 106.9)
- moved C7 77.7 mm to (23.5, 126.7)
- moved C5 62.0 mm to (136.6, 94.7), turned to -90 degrees
- moved C11 50.4 mm to (43.2, 80.1)
- moved C8 47.2 mm to (50.9, 126.6)
- moved C3 5.13 mm to (29.7, 51.6), turned to 90 degrees
- moved C1 1.66 mm to (93.3, 48.7)
- moved C10 0.20 mm to (98.5, 126.0)
- moved C9 0.17 mm to (72.8, 126.7)
Connections:
- U1 pad 34: BTN_NAV2 -> unconnected-(U1-GPIO23-Pad34)
- U1 pad 35: BTN_ADF1 -> unconnected-(U1-GPIO22-Pad35)
- U1 pad 36: unconnected-(U1-EXIO2-Pad36) -> BTN_NAV2
- U1 pad 37: unconnected-(U1-EXIO3-Pad37) -> BTN_ADF1
Routing:
- net +5V: track 469.3 -> 450.3 mm
- net GND: track 89.1 -> 84.7 mm
- net SW3_B: track 65.4 -> 61.6 mm, vias 0 -> 2
- net SW3_A: track 47.8 -> 50.9 mm, vias 0 -> 2
- net BTN_ADF1: track 59.4 -> 61.9 mm
- net BTN_NAV2: track 39.4 -> 41.6 mm
- net LED_DIN: track 43.6 -> 45.1 mm
- net COM2_LED: track 108.8 -> 110.4 mm, vias 5 -> 6
- net +3V3: track 356.2 -> 356.4 mm, vias 4 -> 5
