File: PCBs/Radio Ident/Radio Ident.kicad_sch (KiCad schematic)
At the start: 31 parts, among them SW1 SW_Push, SW2 SW_Push, SW3 SW_Push, SW4 SW_Push, SW5 SW_Push, SW6 SW_Push, U1 XIAO-ESP32-C3-SMD, U3 TYPE-C 6PLCH10.0 073

Commit message: Update drill files and job configuration for radio panel PCBs
- Updated creation dates in NPTH and PTH drill files to 2026-08-13.
- Modified drill sizes for various tool definitions in NPTH and PTH files.
- Added new coordinates for tool paths in PTH drill file.
- Adjusted job configuration file creation date to 2026-08-13.
Parts:
- D7: value D -> 1N5819; footprint Diode_THT:D_DO-41_SOD81_P10.16mm_Horizontal -> Diode_THT:D_DO-41_SOD81_P7.62mm_Horizontal; LCSC (none) -> C110032
Changed lines of the file:
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@@
 			)
 		)
-		(property "Value" "D"
+		(property "Value" "1N5819"
 			(at 64.77 128.27 0)
 			(show_name no)
@@
 			)
 		)
-		(property "Footprint" "Diode_THT:D_DO-41_SOD81_P10.16mm_Horizontal"
+		(property "Footprint" "Diode_THT:D_DO-41_SOD81_P7.62mm_Horizontal"
 			(at 64.77 132.08 0)
 			(hide yes)
@@
 			(at 64.77 132.08 0)
 			(hide yes)
+			(show_name no)
+			(do_not_autoplace no)
+			(effects
+				(font
+					(size 1.27 1.27)
+				)
+			)
+		)
+		(property "LCSC" "C110032"
+			(at 64.77 132.08 0)
+			(hide yes)
