File: PCBs/Radio Panel/learsim pcbs.kicad_pcb (KiCad board)
At the start: 2 copper layers, 120 x 110 mm, 58 parts, among them SW1 MHz, SW2 KHz, SW3 2MD1T1B1M2QES-5, U1 ESP32-C6-DEV-KIT-N8, U2 MAX7219, U3 MAX7219

Commit message: Add new drill files and job configuration for learsim PCBs
- Created non-plated through hole (NPTH) drill file for learsim PCBs.
- Created plated through hole (PTH) drill file for learsim PCBs.
- Added job configuration file for learsim PCBs including specifications and file attributes.
- Updated symbol library table to include new components for the project.
- Modified project settings in .kicad_prl file to adjust active layer and visibility settings.
- Updated project properties in .kicad_pro file to include step file path and cleaned up used designators.
Parts:
- ADF1, COM1, COM2, NAV1, NAV2, Switch1: footprint PCM_Switch_Keyboard_Cherry_MX:SW_Cherry_MX_PCB -> PCM_Switch_Keyboard_Kailh:SW_Kailh_Choc_V2
- moved C6 0.52 mm to (122.4, 106.6)
Routing:
- net BTN_COM2: track 88.8 -> 77.8 mm
- net BTN_NAV1: track 57.6 -> 53.4 mm
- net BTN_Switch1: track 83.2 -> 80.3 mm
- net +3V3: track 356.4 -> 359.2 mm
- net BTN_ADF1: track 61.9 -> 64.2 mm
- net BTN_COM1: track 100.9 -> 98.8 mm
- net GND: track 84.7 -> 85.9 mm
- net BTN_NAV2: track 41.6 -> 42.7 mm

Commit message: Update drill files and job configuration for radio panel PCBs
- Updated creation dates in NPTH and PTH drill files to 2026-08-13.
- Modified drill sizes for various tool definitions in NPTH and PTH files.
- Added new coordinates for tool paths in PTH drill file.
- Adjusted job configuration file creation date to 2026-08-13.
Parts:
- added C19: 10µF, Capacitor_THT:C_Disc_D5.0mm_W2.5mm_P5.00mm, B.Cu at (136.8, 104.0)
- added C20: 0.1µF, Capacitor_THT:C_Disc_D5.0mm_W2.5mm_P5.00mm, F.Cu at (84.1, 44.9)
- added D9: 1N5819, Diode_THT:D_DO-41_SOD81_P7.62mm_Horizontal, F.Cu at (79.6, 44.9)
- added R19: 5.1k, Resistor_THT:R_Axial_DIN0207_L6.3mm_D2.5mm_P7.62mm_Horizontal, B.Cu at (88.8, 41.8)
- added R20: 5.1k, Resistor_THT:R_Axial_DIN0207_L6.3mm_D2.5mm_P7.62mm_Horizontal, B.Cu at (75.5, 34.0)
- added U4: TYPE-C 6PLCH10.0 073, Rotary:USB-C-TH_TYPE-C-6PLCH10.0-073, B.Cu at (82.5, 31.9)
- moved C5 4.41 mm to (136.6, 90.2)
Connections:
- DS1 pad 1: U3_SEG_D -> U3_SEG_F
- DS1 pad 10: U3_SEG_F -> U3_SEG_D
- DS1 pad 11: U3_SEG_A -> U3_SEG_E
- DS1 pad 2: U3_SEG_DP -> U3_SEG_A
- DS1 pad 3: U3_SEG_E -> U3_SEG_B
- DS1 pad 4: U3_SEG_C -> U3_SEG_G
- DS1 pad 5: U3_DIG5 -> U3_DIG3
- DS1 pad 6: U3_SEG_G -> U3_DIG4
- DS1 pad 7: U3_SEG_B -> U3_DIG5
- DS1 pad 8: U3_DIG4 -> U3_SEG_DP
- DS1 pad 9: U3_DIG3 -> U3_SEG_C
- DS2 pad 1: U2_SEG_D -> U2_SEG_F
- DS2 pad 10: U2_SEG_F -> U2_SEG_D
- DS2 pad 11: U2_SEG_A -> U2_SEG_E
- DS2 pad 2: U2_SEG_DP -> U2_SEG_A
- DS2 pad 3: U2_SEG_E -> U2_SEG_B
- DS2 pad 4: U2_SEG_C -> U2_SEG_G
- DS2 pad 5: U2_DIG5 -> U2_DIG3
- DS2 pad 6: U2_SEG_G -> U2_DIG4
- DS2 pad 7: U2_SEG_B -> U2_DIG5
- DS2 pad 8: U2_DIG4 -> U2_SEG_DP
- DS2 pad 9: U2_DIG3 -> U2_SEG_C
Routing:
- net U2_SEG_A: track 14.2 -> 47.9 mm, vias 0 -> 1
- net U2_SEG_F: track 17.9 -> 40.8 mm
- net U2_SEG_B: track 17.1 -> 32.2 mm
- net U2_DIG3: track 24.7 -> 39.8 mm
- net U3_DIG4: track 42.0 -> 56.6 mm, vias 1 -> 0
- net U3_SEG_F: track 11.0 -> 24.6 mm
- net U3_DIG3: track 28.2 -> 41.5 mm
- net U2_SEG_DP: track 18.1 -> 30.9 mm, vias 0 -> 1
- net U3_DIG5: track 38.6 -> 27.3 mm, vias 2 -> 1
- net Net-(D9-A): track 0.00 -> 11.1 mm
- net U3_SEG_DP: track 18.9 -> 27.8 mm, vias 0 -> 1
- net Net-(U4-CC2): track 0.00 -> 7.67 mm
- net U3_SEG_E: track 18.9 -> 11.4 mm
- net Net-(U4-CC1): track 0.00 -> 6.93 mm
- net U2_SEG_G: track 24.6 -> 18.2 mm
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